Commit message: motor commands for points

File: movit_robot_arm_sim/config/gazebo_robot_arm.urdf (robot description, URDF)
Before this commit: robot robot_arm, 6 links, 5 joints
Links:
- link base_link: mass 0.096038 -> 1.0
Joints:
- joint joint_1: limit lower=-1.5708 upper=1.5708 effort=30 velocity=1 -> lower=-1.5708 upper=1.5708 effort=300 velocity=1
- joint joint_2: limit lower=-1.5708 upper=1.5708 effort=30 velocity=1 -> lower=-1.5708 upper=1.5708 effort=300 velocity=1
- joint joint_3: limit lower=-1.5708 upper=1.5708 effort=30 velocity=1 -> lower=-1.5708 upper=1.5708 effort=300 velocity=1
- joint joint_4: limit lower=-1.5708 upper=1.5708 effort=30 velocity=1 -> lower=-1.5708 upper=1.5708 effort=300 velocity=1
